Commit message: 驱动包完成

File: src/02.base/b2_description/urdf/b2_description.urdf (robot description, URDF)
Before this commit: robot b2_description, 37 links, 36 joints
Links:
- added link base_footprint
Joints:
- added joint joint_base: type fixed, parent base_footprint, child base_link, origin xyz=0.0 0.0 0.40 rpy=0.0 0.0 0.0
